File: CurrentSinkOrSwim.kicad_pcb (KiCad board)
At the start: 2 copper layers, 57.1 x 64 mm, 36 parts, among them P1 HEATSINK, P101 CONN_01X02, P102 CONN_01X03, P103 CONN_01X02, Q401 BUK9575, U201 LMV358, U301 LM2931

Commit message: adjusted R303 to get 2.7V, exchanged other parts for availability
Parts:
- Q401: value BUK9575 -> PHP79NQ08LT
- R202: value 9K -> 9.09K
- R303: value 21.6K -> 34K
Changed lines of the file:
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@@
     (links 52)
     (no_connects 0)
-    (area 93.514057 27.4632 160.485943 92.5288)
+    (area 98.374999 28.016999 155.625001 92.125001)
     (thickness 1.6)
     (drawings 8)
@@
       (effects (font (size 1 1) (thickness 0.15)))
     )
-    (fp_text value BUK9575 (at 0 3.81) (layer F.SilkS) hide
+    (fp_text value PHP79NQ08LT (at 0 3.81) (layer F.SilkS) hide
       (effects (font (size 1 1) (thickness 0.15)))
     )
@@
       (effects (font (size 1 1) (thickness 0.15)))
     )
-    (fp_text value 9K (at 0 2.1 270) (layer F.Fab)
+    (fp_text value 9.09K (at 0 2.1 270) (layer F.Fab)
       (effects (font (size 1 1) (thickness 0.15)))
     )
@@
       (effects (font (size 1 1) (thickness 0.15)))
     )
-    (fp_text value 21.6K (at 0 2.1 90) (layer F.Fab)
-      (effects (font (size 1 1) (thickness 0.15)))
-    )
+    (fp_text value 34K (at 0 2.1 90) (layer F.Fab)
+      (effects (font (size 1 1) (thickness 0.15)))
+    )
